File: monitor_lamp_custom_pcb/monitor_lamp_custom_pcb.kicad_pcb (KiCad board)
At the start: 0 parts

Commit message: Added custom library component to the project
In Kicad not all components are present in the default library, some sensors or modules have to be manually added importing symbols and footprint.
Putting this components inside the project is useful so if someone will download it, in is not necessary to search and import the components
Parts:
- added C1: 1µF, Capacitor_SMD:C_0603_1608Metric, F.Cu at (265.8, 23.3)
- added C2: 10uF, Capacitor_SMD:C_1206_3216Metric, F.Cu at (261.8, 37.5)
- added C3: 100nF, Capacitor_SMD:C_0603_1608Metric, F.Cu at (265.8, 25.8)
- added C4: 100nF, Capacitor_SMD:C_0402_1005Metric, F.Cu at (254.5, 43.4)
- added C5: 10uF, Capacitor_SMD:C_1206_3216Metric, F.Cu at (261.8, 40.9)
- added C6: 10uF, Capacitor_SMD:C_0805_2012Metric, F.Cu at (266.8, 37.4)
- added C7: 10uF, Capacitor_SMD:C_0805_2012Metric, F.Cu at (266.8, 40.4)
- added C8: 47uF, Capacitor_SMD:C_1206_3216Metric, F.Cu at (261.8, 44.2)
- added C9: 100nF, Capacitor_SMD:C_0805_2012Metric, F.Cu at (266.8, 43.4)
- added D1: 1N5819WS, Diode_SMD:D_SOD-323, F.Cu at (228.2, 53.6)
- added IC1: HUSB238, Custom_Components:SON50P300X300X80-11N-D, F.Cu at (270.4, 28.9)
- added J2: VEML7700_Connection, Connector_PinHeader_2.54mm:PinHeader_1x04_P2.54mm_Horizontal, F.Cu at (236.3, 24.3)
- added J3: LD2410C_Connection, Connector_PinHeader_2.54mm:PinHeader_1x04_P2.54mm_Horizontal, F.Cu at (236.3, 36.5)
- added J4: Conn_01x02, TerminalBlock_Phoenix:TerminalBlock_Phoenix_PT-1,5-2-5.0-H_1x02_P5.00mm_Horizontal, F.Cu at (237.6, 51.4)
- added L1: 10uH, Inductor_SMD:L_SXN_SMDRI124, F.Cu at (256.6, 28.9)
- added L2: 4.7uH, Inductor_SMD:L_Murata_LQH55DN_5.7x5.0mm, F.Cu at (254.2, 39.1)
- added Q1: AO3401A, Package_TO_SOT_SMD:SOT-23, F.Cu at (270.2, 33.4)
- added Q2: IRLZ44N, Package_TO_SOT_THT:TO-220-3_Vertical, F.Cu at (217.7, 51.5)
- added R1: 10, Resistor_SMD:R_0603_1608Metric, F.Cu at (265.8, 28.3)
- added R10: 10k, Resistor_SMD:R_0402_1005Metric, F.Cu at (270.5, 44.8)
- added R2: 5.1k, Resistor_SMD:R_0402_1005Metric, F.Cu at (270.5, 36.8)
- added R3: 49.9k, Resistor_SMD:R_0402_1005Metric, F.Cu at (270.5, 38.8)
- added R4: 14k, Resistor_SMD:R_0603_1608Metric, F.Cu at (265.8, 30.8)
- added R5: 22, Resistor_SMD:R_0402_1005Metric, F.Cu at (231.8, 53.2)
- added R6: 100k, Resistor_SMD:R_0603_1608Metric, F.Cu at (228.1, 56.4)
- added R7: 140k, Resistor_SMD:R_0402_1005Metric, F.Cu at (270.5, 40.8)
- added R8: 10k, Resistor_SMD:R_0603_1608Metric, F.Cu at (265.8, 33.3)
- added R9: 54.9k, Resistor_SMD:R_0402_1005Metric, F.Cu at (270.5, 42.8)
- added U1: TPS563300, Package_TO_SOT_SMD:SOT-583-8, F.Cu at (251.3, 44.4)
- added U2: TPS561208DDCT, Custom_Components:SOT95P280X110-6N, F.Cu at (270.9, 24.2)
- added U3: ESP32-C3_SUPERMINI_TH, Custom_Sensors:MODULE_ESP32-C3_SUPERMINI_TH, F.Cu at (224.3, 35.4)
- added U4: MAX40200AUK, Package_TO_SOT_SMD:SOT-23-5, F.Cu at (228.6, 50.0)
Other:
- copper layers 0 -> 2
